File: KiCad/CM4_FanCRTL_MAX31740.sch (KiCad schematic (older format))
At the start: 12 parts, among them J16 47053-1000, U5 MAX31740ATA+

Commit message: reworked descriptive text to be more precise
Other:
- note added: "PLEASE READ:\n\nC36: 330 nF for 33Hz; 430nF for 25kHz PWM\n\nD0: PWM duty cycle for temperatures below T_MIN; connect to GND for 0%, to VDD for D_MIN; connecting pad 1 and 2 on jumper JP1 recommended\n\nThermistor voltage devider: configured for T_Start 25°C with finest control range\n\nD_MIN voltage devider: sets minimum active PWM duty cycle (typically between 0.05VDD to 0.2VDD, depending on de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"
- note removed: "PLEASE READ:\n\nCF: 330 nF for 33Hz; 430nF for 25kHz PWM\n\nD0: PWM duty cycle for temperatures below T_MIN; GND for 0%, VDD for D_MIN; connecting pad 1 and 2 on jumper recommended\n\nThermistor voltage devider: configured for T_Start 25°C with finest control range\n\nD_MIN voltage devider: sets minimum active PWM duty cycle (typically between 0.05VDD to 0.2VDD, depending on desired minimum duty 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"
Changed lines of the file:
@@
 $EndComp
 Text Notes 1400 1600 0    50   ~ 0
-PLEASE READ:\n\nCF:    330 nF for 33Hz; 430nF for 25kHz PWM\n\nD0:    PWM duty cycle for temperatures below T_MIN; GND for 0%, VDD for D_MIN; connecting pad 1 and 2 on jumper recommended\n\nThermistor voltage devider: configured for T_Start 25°C with finest control range\n\nD_MIN voltage devider: sets minimum active PWM duty cycle (typically between 0.05VDD to 0.2VDD, depending on desired minimum duty cycle.) with VMIN/VDD = R2/(R1+R2) = DMIN (%)/200
+PLEASE READ:\n\nC36:   330 nF for 33Hz; 430nF for 25kHz PWM\n\nD0:    PWM duty cycle for temperatures below T_MIN; connect to GND for 0%, to VDD for D_MIN; connecting pad 1 and 2 on jumper JP1 recommended\n\nThermistor voltage devider:    configured for T_Start 25°C with finest control range\n\nD_MIN voltage devider:    sets minimum active PWM duty cycle (typically between 0.05VDD to 0.2VDD, depending on desired minimum duty cycle.) with VMIN/VDD = R2/(R1+R2) = DMIN (%)/200
 Wire Wire Line
 	7450 3550 7450 3600
