File: KiCad/CM4_FanCRTL_MAX31740.sch (KiCad schematic (older format))
At the start: 12 parts, among them J16 47053-1000, U5 MAX31740ATA+

Commit message: replaced wrong GND symbol
Connections:
- net labels removed: GNDD
Changed lines of the file:
@@
 Wire Wire Line
 	5950 4450 5950 4650
-$Comp
-L power:GNDD #PWR0156
-U 1 1 5FBC7916
-P 3350 3900
-F 0 "#PWR0156" H 3350 3650 50  0001 C CNN
-F 1 "GNDD" H 3354 3745 50  0000 C CNN
-F 2 "" H 3350 3900 50  0001 C CNN
-F 3 "" H 3350 3900 50  0001 C CNN
-	1    3350 3900
-	1    0    0    -1
-$EndComp
 Wire Wire Line
 	2850 3450 2850 4200
@@
 NoConn ~ 6850 3550
 NoConn ~ 8100 4050
+$Comp
+L power:GND #PWR?
+U 1 1 5FCF77BB
+P 3350 3900
+F 0 "#PWR?" H 3350 3650 50  0001 C CNN
+F 1 "GND" H 3355 3727 50  0000 C CNN
+F 2 "" H 3350 3900 50  0001 C CNN
+F 3 "" H 3350 3900 50  0001 C CNN
+	1    3350 3900
+	1    0    0    -1
+$EndComp
 $EndSCHEMATC

Commit message: updated symbol and footprint of MAX31740
Parts:
- removed U5: MAX31740ATA+, CM4_MATX:MAX31740ATA&plus_, symbol CM4_MATX:MAX31740ATA+
- added U?: MAX31740ATA+, CM4_MATX:MAX31740ATA&plus_, symbol CM4_MATX:MAX31740ATA+
Connections:
- net labels added: D0, DMIN, FREQ, PWM_OUT, SENSE, SLOPE
Changed lines of the file:
@@
 L Device:R R23
 U 1 1 5FBB909F
-P 5950 4800
-F 0 "R23" H 6020 4846 50  0000 L CNN
-F 1 "R5.5k" H 6020 4755 50  0000 L CNN
-F 2 "CM4_MATX:R_0805_2012Metric" V 5880 4800 50  0001 C CNN
-F 3 "~" H 5950 4800 50  0001 C CNN
-	1    5950 4800
+P 5950 4900
+F 0 "R23" H 6020 4946 50  0000 L CNN
+F 1 "R5.5k" H 6020 4855 50  0000 L CNN
+F 2 "CM4_MATX:R_0805_2012Metric" V 5880 4900 50  0001 C CNN
+F 3 "~" H 5950 4900 50  0001 C CNN
+	1    5950 4900
 	1    0    0    -1
 $EndComp
@@
 	5600 4450 5600 4700
 Wire Wire Line
-	5950 4950 5950 5200
-Wire Wire Line
-	5950 4450 5950 4650
+	5950 5050 5950 5300
 Wire Wire Line
 	2850 3450 2850 4200
@@
 Wire Wire Line
 	8000 3600 7450 3600
-Connection ~ 7450 3600
-Wire Wire Line
-	7450 3600 7450 3650
+Wire Wire Line
+	8000 3600 8000 3650
 Wire Wire Line
 	8000 2250 8000 2750
@@
 	6850 3950 8100 3950
 $Comp
-L CM4_MATX:MAX31740ATA+ U5
-U 1 1 5FC49528
-P 4850 2950
-F 0 "U5" H 5850 3337 60  0000 C CNN
-F 1 "MAX31740ATA+" H 5850 3231 60  0000 C CNN
-F 2 "CM4_MATX:MAX31740ATA&plus_" H 5850 3190 60  0001 C CNN
-F 3 "" H 4850 2650 60  0000 C CNN
-	1    4850 2950
-	1    0    0    -1
-$EndComp
-$Comp
-L power:GND #PWR?
+L power:GND #PWR0153
 U 1 1 5FC7838A
 P 2850 4800
-F 0 "#PWR?" H 2850 4550 50  0001 C CNN
+F 0 "#PWR0153" H 2850 4550 50  0001 C CNN
 F 1 "GND" H 2855 4627 50  0000 C CNN
 F 2 "" H 2850 4800 50  0001 C CNN
@@
 $EndComp
 $Comp
-L power:GND #PWR?
+L power:GND #PWR0154
 U 1 1 5FC7888D
 P 5600 4700
-F 0 "#PWR?" H 5600 4450 50  0001 C CNN
+F 0 "#PWR0154" H 5600 4450 50  0001 C CNN
 F 1 "GND" H 5605 4527 50  0000 C CNN
 F 2 "" H 5600 4700 50  0001 C CNN
@@
 $EndComp
 $Comp
-L power:GND #PWR?
+L power:GND #PWR0155
 U 1 1 5FC78D00
-P 5950 5200
-F 0 "#PWR?" H 5950 4950 50  0001 C CNN
-F 1 "GND" H 5955 5027 50  0000 C CNN
-F 2 "" H 5950 5200 50  0001 C CNN
-F 3 "" H 5950 5200 50  0001 C CNN
-	1    5950 5200
-	1    0    0    -1
-$EndComp
-$Comp
-L power:GND #PWR?
+P 5950 5300
+F 0 "#PWR0155" H 5950 5050 50  0001 C CNN
+F 1 "GND" H 5955 5127 50  0000 C CNN
+F 2 "" H 5950 5300 50  0001 C CNN
+F 3 "" H 5950 5300 50  0001 C CNN
+	1    5950 5300
+	1    0    0    -1
+$EndComp
+$Comp
+L power:GND #PWR0156
 U 1 1 5FC78FAF
 P 7950 4400
-F 0 "#PWR?" H 7950 4150 50  0001 C CNN
+F 0 "#PWR0156" H 7950 4150 50  0001 C CNN
 F 1 "GND" H 7955 4227 50  0000 C CNN
 F 2 "" H 7950 4400 50  0001 C CNN
@@
 $EndComp
 $Comp
-L power:GND #PWR?
+L power:GND #PWR0157
 U 1 1 5FC79499
-P 7450 3650
-F 0 "#PWR?" H 7450 3400 50  0001 C CNN
-F 1 "GND" H 7455 3477 50  0000 C CNN
-F 2 "" H 7450 3650 50  0001 C CNN
-F 3 "" H 7450 3650 50  0001 C CNN
-	1    7450 3650
-	1    0    0    -1
-$EndComp
-$Comp
-L power:GND #PWR?
+P 8000 3650
+F 0 "#PWR0157" H 8000 3400 50  0001 C CNN
+F 1 "GND" H 8005 3477 50  0000 C CNN
+F 2 "" H 8000 3650 50  0001 C CNN
+F 3 "" H 8000 3650 50  0001 C CNN
+	1    8000 3650
+	1    0    0    -1
+$EndComp
+$Comp
+L power:GND #PWR0158
 U 1 1 5FC7995C
 P 9000 3250
-F 0 "#PWR?" H 9000 3000 50  0001 C CNN
+F 0 "#PWR0158" H 9000 3000 50  0001 C CNN
 F 1 "GND" H 9005 3077 50  0000 C CNN
 F 2 "" H 9000 3250 50  0001 C CNN
@@
 NoConn ~ 8100 4050
 $Comp
-L power:GND #PWR?
+L power:GND #PWR0159
 U 1 1 5FCF77BB
 P 3350 3900
-F 0 "#PWR?" H 3350 3650 50  0001 C CNN
+F 0 "#PWR0159" H 3350 3650 50  0001 C CNN
 F 1 "GND" H 3355 3727 50  0000 C CNN
 F 2 "" H 3350 3900 50  0001 C CNN
@@
 	1    0    0    -1
 $EndComp
+Text Label 3950 4200 0    50   ~ 0
+DMIN
+Text Label 4550 3450 0    50   ~ 0
+SENSE
+Text Label 7050 2950 0    50   ~ 0
+D0
+Text Label 7050 3150 0    50   ~ 0
+FREQ
+Text Label 7100 3950 0    50   ~ 0
+PWM_OUT
+Connection ~ 8000 3600
+Text Label 5950 4700 1    50   ~ 0
+SLOPE
+Wire Wire Line
+	5950 4450 5950 4750
+$Comp
+L CM4_MATX:MAX31740ATA+ U?
+U 1 1 5FD3336C
+P 4850 2950
+F 0 "U?" H 5850 3337 60  0000 C CNN
+F 1 "MAX31740ATA+" H 5850 3231 60  0000 C CNN
+F 2 "CM4_MATX:MAX31740ATA&plus_" H 5850 3190 60  0001 C CNN
+F 3 "https://datasheets.maximintegrated.com/en/ds/MAX31740.pdf" H 4850 2650 60  0001 C CNN
+F 4 "700-MAX31740ATA+" H 5550 3800 50  0001 C CNN "Mouser No"
+F 5 "Maxim Integrated" H 5500 3700 50  0001 C CNN "Mfr."
+F 6 "MAX31740ATA+" H 5450 3600 50  0001 C CNN "Mfr. No"
+	1    4850 2950
+	1    0    0    -1
+$EndComp

Commit message: updated schematic
Parts:
- gave numbers to parts that had none: 1
Changed lines of the file:
@@
 	5950 4450 5950 4750
 $Comp
-L CM4_MATX:MAX31740ATA+ U?
+L CM4_MATX:MAX31740ATA+ U5
 U 1 1 5FD3336C
 P 4850 2950
-F 0 "U?" H 5850 3337 60  0000 C CNN
+F 0 "U5" H 5850 3337 60  0000 C CNN
 F 1 "MAX31740ATA+" H 5850 3231 60  0000 C CNN
 F 2 "CM4_MATX:MAX31740ATA&plus_" H 5850 3190 60  0001 C CNN
