File: KiCad/CM4_FanCRTL_MAX6615.sch (KiCad schematic (older format))
At the start: 15 parts

Commit message: added net names to schematic
Parts:
- removed U?: MAX6615AEE+, CM4_MATX:MAX6615AEE&plus_, symbol CM4_MATX:MAX6615AEE+
- added U5: MAX6615AEE+, CM4_MATX:MAX6615AEE&plus_, symbol CM4_MATX:MAX6615AEE+
- gave numbers to parts that had none: 14
Connections:
- net labels added: PWM1, PWM2, REF, TACH1, TACH2, TH1, TH2, ~FAN_FAIL, ~OT
Changed lines of the file:
@@
 Comment4 ""
 $EndDescr
-$Comp
-L CM4_MATX:MAX6615AEE+ U?
-U 1 1 5FC85D5A
-P 4850 2350
-F 0 "U?" H 5850 2737 60  0000 C CNN
-F 1 "MAX6615AEE+" H 5850 2631 60  0000 C CNN
-F 2 "CM4_MATX:MAX6615AEE&plus_" H 5850 2590 60  0001 C CNN
-F 3 "https://datasheets.maximintegrated.com/en/ds/MAX6615-MAX6616.pdf" H 4600 900 60  0001 C CNN
-	1    4850 2350
-	1    0    0    -1
-$EndComp
 Text HLabel 3950 1800 0    50   Input ~ 0
 3.3V
@@
 	3950 1800 4550 1800
 $Comp
-L Device:R R?
+L Device:R R19
 U 1 1 5FC8780F
 P 3650 2850
-F 0 "R?" H 3720 2896 50  0000 L CNN
+F 0 "R19" H 3720 2896 50  0000 L CNN
 F 1 "R1.6k" H 3720 2805 50  0000 L CNN
 F 2 "CM4_MATX:R_0805_2012Metric" V 3580 2850 50  0001 C CNN
@@
 $EndComp
 $Comp
-L Device:R R?
+L Device:R R20
 U 1 1 5FC87BE7
 P 3650 3250
-F 0 "R?" H 3720 3296 50  0000 L CNN
+F 0 "R20" H 3720 3296 50  0000 L CNN
 F 1 "R1.6k" H 3720 3205 50  0000 L CNN
 F 2 "CM4_MATX:R_0805_2012Metric" V 3580 3250 50  0001 C CNN
@@
 $EndComp
 $Comp
-L Device:C C?
+L Device:C C35
 U 1 1 5FC87EC1
 P 4150 2850
-F 0 "C?" H 4265 2896 50  0000 L CNN
+F 0 "C35" H 4265 2896 50  0000 L CNN
 F 1 "C100p" H 4265 2805 50  0000 L CNN
 F 2 "CM4_MATX:C_0805_2012Metric" H 4188 2700 50  0001 C CNN
@@
 $EndComp
 $Comp
-L Device:C C?
+L Device:C C36
 U 1 1 5FC881D0
 P 4150 3250
-F 0 "C?" H 4265 3296 50  0000 L CNN
+F 0 "C36" H 4265 3296 50  0000 L CNN
 F 1 "C100p" H 4265 3205 50  0000 L CNN
 F 2 "CM4_MATX:C_0805_2012Metric" H 4188 3100 50  0001 C CNN
@@
 $EndComp
 $Comp
-L Device:R R?
+L Device:R R23
 U 1 1 5FC884AB
 P 7350 2050
-F 0 "R?" H 7280 2004 50  0000 R CNN
+F 0 "R23" H 7280 2004 50  0000 R CNN
 F 1 "R10k" H 7280 2095 50  0000 R CNN
 F 2 "CM4_MATX:R_0805_2012Metric" V 7280 2050 50  0001 C CNN
@@
 $EndComp
 $Comp
-L Device:R R?
+L Device:R R24
 U 1 1 5FC889AE
 P 7750 2050
-F 0 "R?" H 7820 2096 50  0000 L CNN
+F 0 "R24" H 7820 2096 50  0000 L CNN
 F 1 "R10k" H 7820 2005 50  0000 L CNN
 F 2 "CM4_MATX:R_0805_2012Metric" V 7680 2050 50  0001 C CNN
@@
 Connection ~ 3650 3450
 $Comp
-L Device:Thermistor_NTC TH?
+L Device:Thermistor_NTC TH2
 U 1 1 5FC920BC
 P 2900 3850
-F 0 "TH?" H 2998 3896 50  0000 L CNN
+F 0 "TH2" H 2998 3896 50  0000 L CNN
 F 1 "Thermistor_NTC" H 2998 3805 50  0000 L CNN
 F 2 "CM4_MATX:R_0805_2012Metric" H 2900 3900 50  0001 C CNN
@@
 	2500 4150 2500 4400
 $Comp
-L power:GND #PWR?
+L power:GND #PWR0153
 U 1 1 5FC933CA
 P 2500 4400
-F 0 "#PWR?" H 2500 4150 50  0001 C CNN
+F 0 "#PWR0153" H 2500 4150 50  0001 C CNN
 F 1 "GND" H 2505 4227 50  0000 C CNN
 F 2 "" H 2500 4400 50  0001 C CNN
@@
 $EndComp
 $Comp
-L power:GND #PWR?
+L power:GND #PWR0154
 U 1 1 5FC93C44
 P 5350 4550
-F 0 "#PWR?" H 5350 4300 50  0001 C CNN
+F 0 "#PWR0154" H 5350 4300 50  0001 C CNN
 F 1 "GND" H 5355 4377 50  0000 C CNN
 F 2 "" H 5350 4550 50  0001 C CNN
@@
 SCL
 $Comp
-L CM4_MATX:47053-1000 J?
+L CM4_MATX:47053-1000 J16
 U 1 1 5FC9B284
 P 9150 2800
-F 0 "J?" H 9778 2696 50  0000 L CNN
+F 0 "J16" H 9778 2696 50  0000 L CNN
 F 1 "47053-1000" H 9778 2605 50  0000 L CNN
 F 2 "CM4_MATX:470531000" H 9800 2900 50  0001 L CNN
@@
 $EndComp
 $Comp
-L CM4_MATX:47053-1000 J?
+L CM4_MATX:47053-1000 J17
 U 1 1 5FC9BCBA
 P 9150 3500
-F 0 "J?" H 9778 3396 50  0000 L CNN
+F 0 "J17" H 9778 3396 50  0000 L CNN
 F 1 "47053-1000" H 9778 3305 50  0000 L CNN
 F 2 "CM4_MATX:470531000" H 9800 3600 50  0001 L CNN
@@
 	9000 3800 9000 4150
 $Comp
-L power:GND #PWR?
+L power:GND #PWR0155
 U 1 1 5FCA871F
 P 9000 4150
-F 0 "#PWR?" H 9000 3900 50  0001 C CNN
+F 0 "#PWR0155" H 9000 3900 50  0001 C CNN
 F 1 "GND" H 9005 3977 50  0000 C CNN
 F 2 "" H 9000 4150 50  0001 C CNN
@@
 Connection ~ 4550 1800
 $Comp
-L Device:Thermistor_NTC TH?
+L Device:Thermistor_NTC TH1
 U 1 1 5FCBAEC4
 P 2500 3050
-F 0 "TH?" H 2598 3096 50  0000 L CNN
+F 0 "TH1" H 2598 3096 50  0000 L CNN
 F 1 "Thermistor_NTC" H 2598 3005 50  0000 L CNN
 F 2 "CM4_MATX:R_0805_2012Metric" H 2500 3100 50  0001 C CNN
@@
 $EndComp
 $Comp
-L Device:R R?
+L Device:R R25
 U 1 1 5FCBCC96
 P 8450 2550
-F 0 "R?" H 8520 2596 50  0000 L CNN
+F 0 "R25" H 8520 2596 50  0000 L CNN
 F 1 "R10k" H 8520 2505 50  0000 L CNN
 F 2 "CM4_MATX:R_0805_2012Metric" V 8380 2550 50  0001 C CNN
@@
 $EndComp
 $Comp
-L Device:R R?
+L Device:R R26
 U 1 1 5FCBDA8D
 P 8450 3250
-F 0 "R?" H 8520 3296 50  0000 L CNN
+F 0 "R26" H 8520 3296 50  0000 L CNN
 F 1 "R10k" H 8520 3205 50  0000 L CNN
 F 2 "CM4_MATX:R_0805_2012Metric" V 8380 3250 50  0001 C CNN
@@
 	8450 2800 6850 2800
 $Comp
-L Device:R R?
+L Device:R R22
 U 1 1 5FCC41D3
 P 4700 4250
-F 0 "R?" H 4770 4296 50  0000 L CNN
+F 0 "R22" H 4770 4296 50  0000 L CNN
 F 1 "R10k" H 4770 4205 50  0000 L CNN
 F 2 "CM4_MATX:R_0805_2012Metric" V 4630 4250 50  0001 C CNN
@@
 $EndComp
 $Comp
-L Device:R R?
+L Device:R R21
 U 1 1 5FCC54C2
 P 4350 4250
-F 0 "R?" H 4420 4296 50  0000 L CNN
+F 0 "R21" H 4420 4296 50  0000 L CNN
 F 1 "R10k" H 4420 4205 50  0000 L CNN
 F 2 "CM4_MATX:R_0805_2012Metric" V 4280 4250 50  0001 C CNN
@@
 	6350 4450 6150 4450
 Connection ~ 6150 4450
+Text Label 2800 2650 0    50   ~ 0
+TH1
+Text Label 3000 3450 0    50   ~ 0
+TH2
+Text Label 4650 3050 0    50   ~ 0
+REF
+Text Label 7200 2800 0    50   ~ 0
+PWM1
+Text Label 7200 2900 0    50   ~ 0
+TACH1
+Text Label 7200 3500 0    50   ~ 0
+PWM2
+Text Label 7200 3600 0    50   ~ 0
+TACH2
+Text Label 6950 2350 0    50   ~ 0
+~FAN_FAIL
+Text Label 6950 2550 0    50   ~ 0
+~OT
+$Comp
+L CM4_MATX:MAX6615AEE+ U5
+U 1 1 5FD13853
+P 4850 2350
+F 0 "U5" H 5850 2737 60  0000 C CNN
+F 1 "MAX6615AEE+" H 5850 2631 60  0000 C CNN
+F 2 "CM4_MATX:MAX6615AEE&plus_" H 5850 2590 60  0001 C CNN
+F 3 "https://datasheets.maximintegrated.com/en/ds/MAX6615-MAX6616.pdf" H 4600 900 60  0001 C CNN
+	1    4850 2350
+	1    0    0    -1
+$EndComp
 $EndSCHEMATC
