File: KiCad/CM4_PCIe_Switch.sch (KiCad schematic (older format))
At the start: 39 parts, among them IC2 PI7C9X2G404SLBFDE, U4 AP7363-10D

Commit message: Tons of wiring and pin straps for PCI-e Switch
Also re-did some hierarchical labels for JTAG
Parts:
- removed R16, R17, R18: 330, symbol Device:R_Small
- added C? (x6): 10uF, symbol Device:C_Small
- added C?: 100nF, symbol Device:C_Small
- added IC?: M24C04-RMN6TP, SOIC127P600X175-8N, symbol _LibLoader:M24C04-RMN6TP
- added R? (x12): 5.1k, symbol Device:R_Small
- added R? (x25): NC, symbol Device:R_Small
- added R? (x9): 330, symbol Device:R_Small
- added R? (x8): 33, symbol Device:R_Small
- added R? (x8): 49.9, symbol Device:R_Small
- added TP?: STATUS0, symbol Connector:TestPoint_Small
- added TP?: STATUS2, symbol Connector:TestPoint_Small
- added TP?: STATUS1, symbol Connector:TestPoint_Small
- added U?: AP7363-10D, CM4_MATX:TO-252-3_TabPin2, symbol CM4_MATX:AP7363-10D
Connections:
- net labels added: +1.0vSB, CLKQ0_N, CLKQ0_P, CLKQ1_N, CLKQ1_P, CLKQ2_N, CLKQ2_P, CLKQ3_N, CLKQ3_P, DWNRST1_L, DWNRST2_L, DWNRST3_L, EECLK, EEPD, GPIO0, GPIO1, GPIO2, GPIO3, GPIO4, PCIE_SW_SMBCLK, PCIE_SW_SMBDATA, PCIE_SW_TCK, PCIE_SW_TDI, PCIE_SW_TDO, PCIE_SW_TMS, PCIE_SW_TRST_L, PL_512B, PWR_SAV, REFCLKN, REFCLKP, RXPOLINV_DIS, SCAN_EN, SLOTCLK, VC1_EN
- net labels removed: SMBCLK, SMBDATA
- wire segments 207 -> 409
- no-connect marks 22 -> 10
Other:
- note added: "+3.3vSB to +1.0vSB voltage regulator"
- note added: "5.1k pull-up, 330 pull-down"
- note added: "Debug Mode Select"
- note added: "Near to IC2"
- note added: "PCI-e Switch EEPROM"
- note added: "Place resistors near IC2\nClock Output Termination"
- note added: "Strap Pins"
- note added: "Strap Pins (Cont.)"
- note removed: "TODO:\nFinish connecting power\nResearch if SMBus can be implemented"
- moved on the sheet: C25, C26, C27, C28, C30, C31, C33, C34, C42, C43, C46, C47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

Commit message: Added second USB dual-stack header and fixed some library references.
Parts:
- IC3: renamed from IC?; symbol _LibLoader:M24C04-RMN6TP -> CM4_MATX:M24C04-RMN6TP
- gave numbers to parts that had none: 73

Commit message: PCIe Wiring, resistor value adjustments, and a bunch of small ERC fixes.
Parts:
- TP1, TP2, TP3: footprint (none) -> CM4_MATX:TestPoint_Pad_D1.0mm; symbol Connector:TestPoint_Small -> CM4_MATX:TestPoint_Small
Connections:
- net SLOTCLK: now also IC2.33 (SLOTCLK)
Changed lines of the file:
@@
 $Descr A4 11693 8268
 encoding utf-8
-Sheet 11 16
+Sheet 16 16
 Title "CM4_MATX: PCIe Switch"
 Date "2020-12-28"
@@
 	1    0    0    -1
 $EndComp
-Text HLabel 9600 4650 0    50   Input ~ 0
+Text HLabel 9600 4700 0    50   Input ~ 0
 +3.3vSB
 $Comp
@@
 Text Label 8350 4950 2    50   ~ 0
 +3.3v
-Text Label 9600 4650 0    50   ~ 0
-+3.3vSB
-Wire Wire Line
-	9600 4650 9600 4700
 Wire Wire Line
 	9600 4700 9850 4700
@@
 Strap Pins (Cont.)
 $Comp
-L Connector:TestPoint_Small TP2
-U 1 1 616C0607
-P 5300 4950
-F 0 "TP2" H 5348 4996 50  0000 L CNN
-F 1 "STATUS0" H 5348 4905 50  0000 L CNN
-F 2 "" H 5500 4950 50  0001 C CNN
-F 3 "~" H 5500 4950 50  0001 C CNN
-	1    5300 4950
-	1    0    0    -1
-$EndComp
-$Comp
-L Connector:TestPoint_Small TP1
+L CM4_MATX:TestPoint_Small TP1
 U 1 1 616C10C3
 P 5300 4750
 F 0 "TP1" H 5348 4796 50  0000 L CNN
 F 1 "STATUS2" H 5348 4705 50  0000 L CNN
-F 2 "" H 5500 4750 50  0001 C CNN
+F 2 "CM4_MATX:TestPoint_Pad_D1.0mm" H 5500 4750 50  0001 C CNN
 F 3 "~" H 5500 4750 50  0001 C CNN
 	1    5300 4750
 	1    0    0    -1
 $EndComp
-$Comp
-L Connector:TestPoint_Small TP3
-U 1 1 616C1BAE
-P 5700 4850
-F 0 "TP3" H 5748 4896 50  0000 L CNN
-F 1 "STATUS1" H 5748 4805 50  0000 L CNN
-F 2 "" H 5900 4850 50  0001 C CNN
-F 3 "~" H 5900 4850 50  0001 C CNN
-	1    5700 4850
-	1    0    0    -1
-$EndComp
 Wire Wire Line
 	5000 4750 5300 4750
@@
 Text HLabel 1200 4650 0    50   Input ~ 0
 PCIE_SW_SMBDATA
+Text Label 9600 4700 0    50   ~ 0
++3.3vSB
+Text Label 1500 6450 1    50   ~ 0
+SLOTCLK
+Wire Wire Line
+	1500 6450 1500 6150
+$Comp
+L CM4_MATX:TestPoint_Small TP3
+U 1 1 616C1BAE
+P 5700 4850
+F 0 "TP3" H 5748 4896 50  0000 L CNN
+F 1 "STATUS1" H 5748 4805 50  0000 L CNN
+F 2 "CM4_MATX:TestPoint_Pad_D1.0mm" H 5900 4850 50  0001 C CNN
+F 3 "~" H 5900 4850 50  0001 C CNN
+	1    5700 4850
+	1    0    0    -1
+$EndComp
+$Comp
+L CM4_MATX:TestPoint_Small TP2
+U 1 1 616C0607
+P 5300 4950
+F 0 "TP2" H 5348 4996 50  0000 L CNN
+F 1 "STATUS0" H 5348 4905 50  0000 L CNN
+F 2 "CM4_MATX:TestPoint_Pad_D1.0mm" H 5500 4950 50  0001 C CNN
+F 3 "~" H 5500 4950 50  0001 C CNN
+	1    5300 4950
+	1    0    0    -1
+$EndComp
 $EndSCHEMATC

Commit message: Started picking passive components, overhauled library
Cleaned up a bunch of schematic library references.
Added datasheets, descriptions for a lot of existing parts.
Picked most capacitor parts, still a couple left.
Cleaned up a fair few footprint references.
Parts:
- C25, C26, C27, C41, C48, C51, C71, C72, C73, C75, C76, C77: footprint (none) -> CM4_MATX:C_0603_1608Metric_Pad1.08x0.95mm_HandSolder; symbol Device:C_Small -> CM4_MATX:C_Small; Description (none) -> 6.3V 10uF X5R 0603 20% Tol; Mfr. (none) -> Samsung; Mfr. No (none) -> CL10A106MQ8NNNC; Mouser Part Number (none) -> 187-CL10A106MQ8NNNC; Mouser Price/Stock (none) -> https://www.mouser.co.uk/ProductDetail/Samsung-Electro-Mech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
- C28, C29, C30, C31, C32, C33, C34, C40, C42, C43, C44, C45, C46, C47, C49, C50, C52, C53, C54, C55, C56, C57, C58, C59, C60, C61, C74: footprint (none) -> CM4_MATX:C_0402_1005Metric_Pad0.74x0.62mm_HandSolder; symbol Device:C_Small -> CM4_MATX:C_Small; Description (none) -> 10V 0.1uF X5R 0402 20% Tol; Mfr. (none) -> AVX; Mfr. No (none) -> 0402ZD104MAT4A; Mouser Part Number (none) -> 581-0402ZD104MAT4A; Mouser Price/Stock (none) -> https://www.mouser.co.uk/ProductDetail/AVX/0402ZD104MAT4A/?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
- IC2: Height 1.6 -> (none); Manufacturer_Name Diodes Inc. -> (none); Manufacturer_Part_Number PI7C9X2G404SLBFDE -> (none); Mfr. (none) -> Diodes Inc.; Mfr. No (none) -> PI7C9X2G404SLBFDE
- IC3: footprint SOIC127P600X175-8N -> CM4_MATX:SOIC127P600X175-8N; Height 1.75 -> (none); Manufacturer_Name STMicroelectronics -> (none); Manufacturer_Part_Number M24C04-RMN6TP -> (none); Mfr. (none) -> STMicroelectronics; Mfr. No (none) -> M24C04-RMN6TP
- R1, R14, R15, R16, R17, R18, R2, R36, R37, R38, R39, R40, R41, R42, R43, R44, R45, R46, R47, R48, R49, R50, R51, R52, R53, R54, R55, R56, R57, R58, R59, R60, R61, R62, R63, R64, R65, R66, R67, R68, R69, R70, R71, R72, R73, R74, R75, R76, R77, R78, R79, R80, R81, R82, R83, R84, R85, R86, R87, R88, R89, R90, R91, R92: symbol Device:R_Small -> CM4_MATX:R_Small
- TP1: Description (none) -> PCIE Port Status 1 Testing Point
- TP2: Description (none) -> PCIE Port Status 2 Testing Point
- TP3: Description (none) -> PCIE Port Status 3 Testing Point
- U19, U4: Description (none) -> LDO Voltage Regulators 1.5A Fast Transient Ultra-LDO Linear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; Mfr. (none) -> Diodes Inc.; Mfr. No (none) -> AP7363-10D-13; Mouser Part Number (none) -> 621-AP7363-10D-13; Mouser Price/Stock (none) -> https://www.mouser.co.uk/ProductDetail/Diodes-Incorporated/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
