File: KiCad/_autosave-CM4_PCIe_Switch.sch (KiCad schematic (older format))
At the start: 90 parts, among them IC2 PI7C9X2G404SLBFDE, IC3 M24C04-RMN6TP, U19 AP7363-10D, U4 AP7363-10D

Commit message: More BOM detailing and small changes
Removed some NC components from the PCI-e subsection
Picked resistor footprints
Picked resistor items in the BOM
Parts:
- R36, R37, R38, R39, R40: footprint (none) -> CM4_MATX:R_0402_1005Metric_Pad0.72x0.64mm_HandSolder; Description (none) -> 0402 1/16W 330Ohm 1%; Mfr. (none) -> Vishay / Dale; Mfr. No (none) -> CRCW0402330RFKEDC; Mouser Part Number (none) -> 71-CRCW0402330RFKEDC; Mouser Price/Stock (none) -> https://www.mouser.co.uk/ProductDetail/Vishay-Dale/CRCW0402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
Changed lines of the file:
@@
 F 0 "R40" V 1650 7300 50  0000 C CNN
 F 1 "330" V 1650 7600 50  0000 C CNN
-F 2 "" H 1700 7450 50  0001 C CNN
-F 3 "~" H 1700 7450 50  0001 C CNN
+F 2 "CM4_MATX:R_0402_1005Metric_Pad0.72x0.64mm_HandSolder" H 1700 7450 50  0001 C CNN
+F 3 "https://www.mouser.co.uk/datasheet/2/427/dcrcwe3-1762152.pdf" H 1700 7450 50  0001 C CNN
+F 4 "0402 1/16W 330Ohm 1%" H 1700 7450 50  0001 C CNN "Description"
+F 5 "Vishay / Dale" H 1700 7450 50  0001 C CNN "Mfr."
+F 6 "CRCW0402330RFKEDC" H 1700 7450 50  0001 C CNN "Mfr. No"
+F 7 "71-CRCW0402330RFKEDC" H 1700 7450 50  0001 C CNN "Mouser Part Number"
+F 8 "https://www.mouser.co.uk/ProductDetail/Vishay-Dale/CRCW0402330RFKEDC/?qs=sGAEpiMZZMvdGkrng054t0DrEhLhGh8gUyDGo38wXjAq0Lll9pYo4A%3D%3D" H 1700 7450 50  0001 C CNN "Mouser Price/Stock"
 	1    1700 7450
 	0    1    1    0
@@
 F 0 "R38" V 1650 7100 50  0000 C CNN
 F 1 "330" V 1650 7400 50  0000 C CNN
-F 2 "" H 1700 7250 50  0001 C CNN
-F 3 "~" H 1700 7250 50  0001 C CNN
+F 2 "CM4_MATX:R_0402_1005Metric_Pad0.72x0.64mm_HandSolder" H 1700 7250 50  0001 C CNN
+F 3 "https://www.mouser.co.uk/datasheet/2/427/dcrcwe3-1762152.pdf" H 1700 7250 50  0001 C CNN
+F 4 "0402 1/16W 330Ohm 1%" H 1700 7250 50  0001 C CNN "Description"
+F 5 "Vishay / Dale" H 1700 7250 50  0001 C CNN "Mfr."
+F 6 "CRCW0402330RFKEDC" H 1700 7250 50  0001 C CNN "Mfr. No"
+F 7 "71-CRCW0402330RFKEDC" H 1700 7250 50  0001 C CNN "Mouser Part Number"
+F 8 "https://www.mouser.co.uk/ProductDetail/Vishay-Dale/CRCW0402330RFKEDC/?qs=sGAEpiMZZMvdGkrng054t0DrEhLhGh8gUyDGo38wXjAq0Lll9pYo4A%3D%3D" H 1700 7250 50  0001 C CNN "Mouser Price/Stock"
 	1    1700 7250
 	0    1    1    0
@@
 F 0 "R39" V 1650 7200 50  0000 C CNN
 F 1 "330" V 1650 7500 50  0000 C CNN
-F 2 "" H 1700 7350 50  0001 C CNN
-F 3 "~" H 1700 7350 50  0001 C CNN
+F 2 "CM4_MATX:R_0402_1005Metric_Pad0.72x0.64mm_HandSolder" H 1700 7350 50  0001 C CNN
+F 3 "https://www.mouser.co.uk/datasheet/2/427/dcrcwe3-1762152.pdf" H 1700 7350 50  0001 C CNN
+F 4 "0402 1/16W 330Ohm 1%" H 1700 7350 50  0001 C CNN "Description"
+F 5 "Vishay / Dale" H 1700 7350 50  0001 C CNN "Mfr."
+F 6 "CRCW0402330RFKEDC" H 1700 7350 50  0001 C CNN "Mfr. No"
+F 7 "71-CRCW0402330RFKEDC" H 1700 7350 50  0001 C CNN "Mouser Part Number"
+F 8 "https://www.mouser.co.uk/ProductDetail/Vishay-Dale/CRCW0402330RFKEDC/?qs=sGAEpiMZZMvdGkrng054t0DrEhLhGh8gUyDGo38wXjAq0Lll9pYo4A%3D%3D" H 1700 7350 50  0001 C CNN "Mouser Price/Stock"
 	1    1700 7350
 	0    1    1    0
@@
 F 0 "R37" V 1650 7000 50  0000 C CNN
 F 1 "330" V 1650 7300 50  0000 C CNN
-F 2 "" H 1700 7150 50  0001 C CNN
-F 3 "~" H 1700 7150 50  0001 C CNN
+F 2 "CM4_MATX:R_0402_1005Metric_Pad0.72x0.64mm_HandSolder" H 1700 7150 50  0001 C CNN
+F 3 "https://www.mouser.co.uk/datasheet/2/427/dcrcwe3-1762152.pdf" H 1700 7150 50  0001 C CNN
+F 4 "0402 1/16W 330Ohm 1%" H 1700 7150 50  0001 C CNN "Description"
+F 5 "Vishay / Dale" H 1700 7150 50  0001 C CNN "Mfr."
+F 6 "CRCW0402330RFKEDC" H 1700 7150 50  0001 C CNN "Mfr. No"
+F 7 "71-CRCW0402330RFKEDC" H 1700 7150 50  0001 C CNN "Mouser Part Number"
+F 8 "https://www.mouser.co.uk/ProductDetail/Vishay-Dale/CRCW0402330RFKEDC/?qs=sGAEpiMZZMvdGkrng054t0DrEhLhGh8gUyDGo38wXjAq0Lll9pYo4A%3D%3D" H 1700 7150 50  0001 C CNN "Mouser Price/Stock"
 	1    1700 7150
 	0    1    1    0
@@
 F 0 "R36" V 1650 6900 50  0000 C CNN
 F 1 "330" V 1650 7200 50  0000 C CNN
-F 2 "" H 1700 7050 50  0001 C CNN
-F 3 "~" H 1700 7050 50  0001 C CNN
+F 2 "CM4_MATX:R_0402_1005Metric_Pad0.72x0.64mm_HandSolder" H 1700 7050 50  0001 C CNN
+F 3 "https://www.mouser.co.uk/datasheet/2/427/dcrcwe3-1762152.pdf" H 1700 7050 50  0001 C CNN
+F 4 "0402 1/16W 330Ohm 1%" H 1700 7050 50  0001 C CNN "Description"
+F 5 "Vishay / Dale" H 1700 7050 50  0001 C CNN "Mfr."
+F 6 "CRCW0402330RFKEDC" H 1700 7050 50  0001 C CNN "Mfr. No"
+F 7 "71-CRCW0402330RFKEDC" H 1700 7050 50  0001 C CNN "Mouser Part Number"
+F 8 "https://www.mouser.co.uk/ProductDetail/Vishay-Dale/CRCW0402330RFKEDC/?qs=sGAEpiMZZMvdGkrng054t0DrEhLhGh8gUyDGo38wXjAq0Lll9pYo4A%3D%3D" H 1700 7050 50  0001 C CNN "Mouser Price/Stock"
 	1    1700 7050
 	0    1    1    0
