File: KiCad/CM4_USB2_Power.sch (KiCad schematic (older format))
At the start: 22 parts, among them U10 MIC2019YM6-TR, U11 MIC2019YM6-TR, U12 MIC2019YM6-TR, U13 MIC2019YM6-TR, U14 MIC2019YM6-TR, U15 MIC2019YM6-TR, U16 MIC2019YM6-TR

Commit message: Started picking passive components, overhauled library
Cleaned up a bunch of schematic library references.
Added datasheets, descriptions for a lot of existing parts.
Picked most capacitor parts, still a couple left.
Cleaned up a fair few footprint references.
Parts:
- C18: footprint (none) -> CM4_MATX:C_1206_3216Metric_Pad1.33x1.80mm_HandSolder; symbol Device:C_Small -> CM4_MATX:C_Small; Description (none) -> 6.3V 100uF X5R 1206 20% Tol; Mfr. (none) -> Samsung; Mfr. No (none) -> CL31A107MQHNNWE; Mouser Part Number (none) -> 187-CL31A107MQHNNWE; Mouser Price/Stock (none) -> https://www.mouser.co.uk/ProductDetail/Samsung-Electro-Mech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
- C20, C22, C24, C35, C36, C37, C38: footprint (none) -> CM4_MATX:C_0603_1608Metric_Pad1.08x0.95mm_HandSolder; symbol Device:C_Small -> CM4_MATX:C_Small; Description (none) -> 6.3V 10uF X5R 0603 20% Tol; Mfr. (none) -> Samsung; Mfr. No (none) -> CL10A106MQ8NNNC; Mouser Part Number (none) -> 187-CL10A106MQ8NNNC; Mouser Price/Stock (none) -> https://www.mouser.co.uk/ProductDetail/Samsung-Electro-Mech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
- R23, R24, R25, R26, R27, R28, R29: symbol Device:R_Small -> CM4_MATX:R_Small
- U10, U11, U12, U13, U14, U15, U16: Height 1.45 -> (none); Manufacturer_Name Microchip -> (none); Manufacturer_Part_Number MIC2019YM6-TR -> (none); Mfr. (none) -> Microchip; Mfr. No (none) -> MIC2019YM6-TR

Commit message: More BOM detailing and small changes
Removed some NC components from the PCI-e subsection
Picked resistor footprints
Picked resistor items in the BOM
Parts:
- R23, R24, R25, R26, R27, R28, R29: footprint (none) -> CM4_MATX:R_0402_1005Metric_Pad0.72x0.64mm_HandSolder; Description (none) -> 0402 1/16W 143Ohm 1%; Mfr. (none) -> Vishay / Dale; Mfr. No (none) -> CRCW0402143RFKEDC; Mouser Part Number (none) -> 71-CRCW0402143RFKEDC; Mouser Price/Stock (none) -> https://www.mouser.co.uk/ProductDetail/Vishay-Dale/CRCW0402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
Changed lines of the file:
@@
 F 0 "R23" H 2359 2596 50  0000 L CNN
 F 1 "143 1%" H 2359 2505 50  0000 L CNN
-F 2 "" H 2300 2550 50  0001 C CNN
-F 3 "~" H 2300 2550 50  0001 C CNN
+F 2 "CM4_MATX:R_0402_1005Metric_Pad0.72x0.64mm_HandSolder" H 2300 2550 50  0001 C CNN
+F 3 "https://www.mouser.co.uk/datasheet/2/427/crcwce3-1762584.pdf" H 2300 2550 50  0001 C CNN
+F 4 "0402 1/16W 143Ohm 1%" H 2300 2550 50  0001 C CNN "Description"
+F 5 "Vishay / Dale" H 2300 2550 50  0001 C CNN "Mfr."
+F 6 "CRCW0402143RFKEDC" H 2300 2550 50  0001 C CNN "Mfr. No"
+F 7 "71-CRCW0402143RFKEDC" H 2300 2550 50  0001 C CNN "Mouser Part Number"
+F 8 "https://www.mouser.co.uk/ProductDetail/Vishay-Dale/CRCW0402143RFKEDC/?qs=sGAEpiMZZMvdGkrng054t0DrEhLhGh8gVrzzIF%252BS5CurukA28nIrVg%3D%3D" H 2300 2550 50  0001 C CNN "Mouser Price/Stock"
 	1    2300 2550
 	1    0    0    -1
@@
 F 0 "R24" H 2359 3596 50  0000 L CNN
 F 1 "143 1%" H 2359 3505 50  0000 L CNN
-F 2 "" H 2300 3550 50  0001 C CNN
-F 3 "~" H 2300 3550 50  0001 C CNN
+F 2 "CM4_MATX:R_0402_1005Metric_Pad0.72x0.64mm_HandSolder" H 2300 3550 50  0001 C CNN
+F 3 "https://www.mouser.co.uk/datasheet/2/427/crcwce3-1762584.pdf" H 2300 3550 50  0001 C CNN
+F 4 "0402 1/16W 143Ohm 1%" H 2300 3550 50  0001 C CNN "Description"
+F 5 "Vishay / Dale" H 2300 3550 50  0001 C CNN "Mfr."
+F 6 "CRCW0402143RFKEDC" H 2300 3550 50  0001 C CNN "Mfr. No"
+F 7 "71-CRCW0402143RFKEDC" H 2300 3550 50  0001 C CNN "Mouser Part Number"
+F 8 "https://www.mouser.co.uk/ProductDetail/Vishay-Dale/CRCW0402143RFKEDC/?qs=sGAEpiMZZMvdGkrng054t0DrEhLhGh8gVrzzIF%252BS5CurukA28nIrVg%3D%3D" H 2300 3550 50  0001 C CNN "Mouser Price/Stock"
 	1    2300 3550
 	1    0    0    -1
@@
 F 0 "R25" H 4309 2596 50  0000 L CNN
 F 1 "143 1%" H 4309 2505 50  0000 L CNN
-F 2 "" H 4250 2550 50  0001 C CNN
-F 3 "~" H 4250 2550 50  0001 C CNN
+F 2 "CM4_MATX:R_0402_1005Metric_Pad0.72x0.64mm_HandSolder" H 4250 2550 50  0001 C CNN
+F 3 "https://www.mouser.co.uk/datasheet/2/427/crcwce3-1762584.pdf" H 4250 2550 50  0001 C CNN
+F 4 "0402 1/16W 143Ohm 1%" H 4250 2550 50  0001 C CNN "Description"
+F 5 "Vishay / Dale" H 4250 2550 50  0001 C CNN "Mfr."
+F 6 "CRCW0402143RFKEDC" H 4250 2550 50  0001 C CNN "Mfr. No"
+F 7 "71-CRCW0402143RFKEDC" H 4250 2550 50  0001 C CNN "Mouser Part Number"
+F 8 "https://www.mouser.co.uk/ProductDetail/Vishay-Dale/CRCW0402143RFKEDC/?qs=sGAEpiMZZMvdGkrng054t0DrEhLhGh8gVrzzIF%252BS5CurukA28nIrVg%3D%3D" H 4250 2550 50  0001 C CNN "Mouser Price/Stock"
 	1    4250 2550
 	1    0    0    -1
@@
 F 0 "R26" H 4309 3596 50  0000 L CNN
 F 1 "143 1%" H 4309 3505 50  0000 L CNN
-F 2 "" H 4250 3550 50  0001 C CNN
-F 3 "~" H 4250 3550 50  0001 C CNN
+F 2 "CM4_MATX:R_0402_1005Metric_Pad0.72x0.64mm_HandSolder" H 4250 3550 50  0001 C CNN
+F 3 "https://www.mouser.co.uk/datasheet/2/427/crcwce3-1762584.pdf" H 4250 3550 50  0001 C CNN
+F 4 "0402 1/16W 143Ohm 1%" H 4250 3550 50  0001 C CNN "Description"
+F 5 "Vishay / Dale" H 4250 3550 50  0001 C CNN "Mfr."
+F 6 "CRCW0402143RFKEDC" H 4250 3550 50  0001 C CNN "Mfr. No"
+F 7 "71-CRCW0402143RFKEDC" H 4250 3550 50  0001 C CNN "Mouser Part Number"
+F 8 "https://www.mouser.co.uk/ProductDetail/Vishay-Dale/CRCW0402143RFKEDC/?qs=sGAEpiMZZMvdGkrng054t0DrEhLhGh8gVrzzIF%252BS5CurukA28nIrVg%3D%3D" H 4250 3550 50  0001 C CNN "Mouser Price/Stock"
 	1    4250 3550
 	1    0    0    -1
@@
 F 0 "R27" H 6259 2596 50  0000 L CNN
 F 1 "143 1%" H 6259 2505 50  0000 L CNN
-F 2 "" H 6200 2550 50  0001 C CNN
-F 3 "~" H 6200 2550 50  0001 C CNN
+F 2 "CM4_MATX:R_0402_1005Metric_Pad0.72x0.64mm_HandSolder" H 6200 2550 50  0001 C CNN
+F 3 "https://www.mouser.co.uk/datasheet/2/427/crcwce3-1762584.pdf" H 6200 2550 50  0001 C CNN
+F 4 "0402 1/16W 143Ohm 1%" H 6200 2550 50  0001 C CNN "Description"
+F 5 "Vishay / Dale" H 6200 2550 50  0001 C CNN "Mfr."
+F 6 "CRCW0402143RFKEDC" H 6200 2550 50  0001 C CNN "Mfr. No"
+F 7 "71-CRCW0402143RFKEDC" H 6200 2550 50  0001 C CNN "Mouser Part Number"
+F 8 "https://www.mouser.co.uk/ProductDetail/Vishay-Dale/CRCW0402143RFKEDC/?qs=sGAEpiMZZMvdGkrng054t0DrEhLhGh8gVrzzIF%252BS5CurukA28nIrVg%3D%3D" H 6200 2550 50  0001 C CNN "Mouser Price/Stock"
 	1    6200 2550
 	1    0    0    -1
@@
 F 0 "R29" H 8209 2596 50  0000 L CNN
 F 1 "143 1%" H 8209 2505 50  0000 L CNN
-F 2 "" H 8150 2550 50  0001 C CNN
-F 3 "~" H 8150 2550 50  0001 C CNN
+F 2 "CM4_MATX:R_0402_1005Metric_Pad0.72x0.64mm_HandSolder" H 8150 2550 50  0001 C CNN
+F 3 "https://www.mouser.co.uk/datasheet/2/427/crcwce3-1762584.pdf" H 8150 2550 50  0001 C CNN
+F 4 "0402 1/16W 143Ohm 1%" H 8150 2550 50  0001 C CNN "Description"
+F 5 "Vishay / Dale" H 8150 2550 50  0001 C CNN "Mfr."
+F 6 "CRCW0402143RFKEDC" H 8150 2550 50  0001 C CNN "Mfr. No"
+F 7 "71-CRCW0402143RFKEDC" H 8150 2550 50  0001 C CNN "Mouser Part Number"
+F 8 "https://www.mouser.co.uk/ProductDetail/Vishay-Dale/CRCW0402143RFKEDC/?qs=sGAEpiMZZMvdGkrng054t0DrEhLhGh8gVrzzIF%252BS5CurukA28nIrVg%3D%3D" H 8150 2550 50  0001 C CNN "Mouser Price/Stock"
 	1    8150 2550
 	1    0    0    -1
@@
 F 0 "R28" H 6259 3596 50  0000 L CNN
 F 1 "143 1%" H 6259 3505 50  0000 L CNN
-F 2 "" H 6200 3550 50  0001 C CNN
-F 3 "~" H 6200 3550 50  0001 C CNN
+F 2 "CM4_MATX:R_0402_1005Metric_Pad0.72x0.64mm_HandSolder" H 6200 3550 50  0001 C CNN
+F 3 "https://www.mouser.co.uk/datasheet/2/427/crcwce3-1762584.pdf" H 6200 3550 50  0001 C CNN
+F 4 "0402 1/16W 143Ohm 1%" H 6200 3550 50  0001 C CNN "Description"
+F 5 "Vishay / Dale" H 6200 3550 50  0001 C CNN "Mfr."
+F 6 "CRCW0402143RFKEDC" H 6200 3550 50  0001 C CNN "Mfr. No"
+F 7 "71-CRCW0402143RFKEDC" H 6200 3550 50  0001 C CNN "Mouser Part Number"
+F 8 "https://www.mouser.co.uk/ProductDetail/Vishay-Dale/CRCW0402143RFKEDC/?qs=sGAEpiMZZMvdGkrng054t0DrEhLhGh8gVrzzIF%252BS5CurukA28nIrVg%3D%3D" H 6200 3550 50  0001 C CNN "Mouser Price/Stock"
 	1    6200 3550
 	1    0    0    -1
