File: KiCad/CM4_GPIO.sch (KiCad schematic (older format))
At the start: 17 parts, among them J16 GSD090012SEU, J17 Conn_02x04_Odd_Even, J18 ARJM11C7-502-AB-ER2-T, J19 Conn_02x20_Odd_Even, J2 CM4_A, J20 Conn_02x04_Odd_Even, U6 74LVC1G07GW, U7 TPD4EUSB30, U8 RT9742GGJ5, U9 TPD4EUSB30

Commit message: Connected all grounds in the schematic and planes
Planes:
In 1 - Ground
In 2 - 3.3v Zone which excludes the IO and 5v Zone around only the IO
Parts:
- added GND (x13): GND, symbol CM4_MATX:GND
Connections:
- net GND: now also GND.1 (GND), GND.1 (GND), GND.1 (GND), GND.1 (GND), GND.1 (GND), GND.1 (GND), GND.1 (GND), GND.1 (GND), GND.1 (GND), GND.1 (GND), GND.1 (GND), GND.1 (GND), GND.1 (GND)
Changed lines of the file:
@@
 	1550 1150 1600 1150
 $Comp
-L CM4_MATX:GND #PWR0154
+L CM4_MATX:GND GND
 U 1 1 5FBDF547
 P 1550 6450
-F 0 "#PWR0154" H 1550 6200 50  0001 C CNN
+F 0 "GND" H 1550 6200 50  0001 C CNN
 F 1 "GND" H 1555 6277 50  0000 C CNN
 F 2 "" H 1550 6450 50  0001 C CNN
@@
 $EndComp
 $Comp
-L CM4_MATX:GND #PWR0155
+L CM4_MATX:GND GND
 U 1 1 5FBDF723
 P 4050 6450
-F 0 "#PWR0155" H 4050 6200 50  0001 C CNN
+F 0 "GND" H 4050 6200 50  0001 C CNN
 F 1 "GND" H 4055 6277 50  0000 C CNN
 F 2 "" H 4050 6450 50  0001 C CNN
@@
 BT_nDis
 $Comp
-L CM4_MATX:GND #PWR0156
+L CM4_MATX:GND GND
 U 1 1 5FC3C044
 P 11000 1150
-F 0 "#PWR0156" H 11000 900 50  0001 C CNN
+F 0 "GND" H 11000 900 50  0001 C CNN
 F 1 "GND" H 11005 977 50  0000 C CNN
 F 2 "" H 11000 1150 50  0001 C CNN
@@
 	9400 950  9400 1350
 $Comp
-L CM4_MATX:GND #PWR0157
+L CM4_MATX:GND GND
 U 1 1 5FD6485E
 P 9400 2700
-F 0 "#PWR0157" H 9400 2450 50  0001 C CNN
+F 0 "GND" H 9400 2450 50  0001 C CNN
 F 1 "GND" H 9405 2527 50  0000 C CNN
 F 2 "" H 9400 2700 50  0001 C CNN
@@
 $EndComp
 $Comp
-L CM4_MATX:GND #PWR0158
+L CM4_MATX:GND GND
 U 1 1 5FD64BC0
 P 8800 2700
-F 0 "#PWR0158" H 8800 2450 50  0001 C CNN
+F 0 "GND" H 8800 2450 50  0001 C CNN
 F 1 "GND" H 8805 2527 50  0000 C CNN
 F 2 "" H 8800 2700 50  0001 C CNN
@@
 	11100 3700 10800 3700
 $Comp
-L CM4_MATX:GND #PWR0159
+L CM4_MATX:GND GND
 U 1 1 5FE636FC
 P 10300 4100
-F 0 "#PWR0159" H 10300 3850 50  0001 C CNN
+F 0 "GND" H 10300 3850 50  0001 C CNN
 F 1 "GND" H 10305 3927 50  0000 C CNN
 F 2 "" H 10300 4100 50  0001 C CNN
@@
 	7850 3500 8150 3500
 $Comp
-L CM4_MATX:GND #PWR0160
+L CM4_MATX:GND GND
 U 1 1 5FEADA78
 P 8650 4100
-F 0 "#PWR0160" H 8650 3850 50  0001 C CNN
+F 0 "GND" H 8650 3850 50  0001 C CNN
 F 1 "GND" H 8655 3927 50  0000 C CNN
 F 2 "" H 8650 4100 50  0001 C CNN
@@
 $EndComp
 $Comp
-L CM4_MATX:GND #PWR0161
+L CM4_MATX:GND GND
 U 1 1 5FFAE3C1
 P 8350 5700
-F 0 "#PWR0161" H 8350 5450 50  0001 C CNN
+F 0 "GND" H 8350 5450 50  0001 C CNN
 F 1 "GND" H 8355 5527 50  0000 C CNN
 F 2 "" H 8350 5700 50  0001 C CNN
@@
 +3.3v
 $Comp
-L CM4_MATX:GND #PWR0162
+L CM4_MATX:GND GND
 U 1 1 600BCD87
 P 10050 5850
-F 0 "#PWR0162" H 10050 5600 50  0001 C CNN
+F 0 "GND" H 10050 5600 50  0001 C CNN
 F 1 "GND" H 10055 5677 50  0000 C CNN
 F 2 "" H 10050 5850 50  0001 C CNN
@@
 	10150 2050 10150 2200
 $Comp
-L CM4_MATX:GND #PWR0163
+L CM4_MATX:GND GND
 U 1 1 601CB73E
 P 10150 2200
-F 0 "#PWR0163" H 10150 1950 50  0001 C CNN
+F 0 "GND" H 10150 1950 50  0001 C CNN
 F 1 "GND" H 10155 2027 50  0000 C CNN
 F 2 "" H 10150 2200 50  0001 C CNN
@@
 	6550 1300 6550 1650
 $Comp
-L CM4_MATX:GND #PWR0165
+L CM4_MATX:GND GND
 U 1 1 603220D6
 P 6550 1650
-F 0 "#PWR0165" H 6550 1400 50  0001 C CNN
+F 0 "GND" H 6550 1400 50  0001 C CNN
 F 1 "GND" H 6555 1477 50  0000 C CNN
 F 2 "" H 6550 1650 50  0001 C CNN
@@
 	7900 1400 7900 1650
 $Comp
-L CM4_MATX:GND #PWR0166
+L CM4_MATX:GND GND
 U 1 1 60363EE2
 P 7900 1650
-F 0 "#PWR0166" H 7900 1400 50  0001 C CNN
+F 0 "GND" H 7900 1400 50  0001 C CNN
 F 1 "GND" H 7905 1477 50  0000 C CNN
 F 2 "" H 7900 1650 50  0001 C CNN
@@
 FP_PLED
 $Comp
-L CM4_MATX:GND #PWR0168
+L CM4_MATX:GND GND
 U 1 1 6054E589
 P 7600 3750
-F 0 "#PWR0168" H 7600 3500 50  0001 C CNN
+F 0 "GND" H 7600 3500 50  0001 C CNN
 F 1 "GND" H 7605 3577 50  0000 C CNN
 F 2 "" H 7600 3750 50  0001 C CNN
